Commit message: Ignition Gazebo用のKobukiの差動駆動のプラグインとros2_controlに入れ替えた．

File: kobuki_description/urdf/kobuki_gazebo.urdf.xacro (robot description, xacro)
@@ -144,22 +144,34 @@
       </sensor>
 	  </gazebo>
-	  <gazebo>
-      <plugin
-        filename="libignition-gazebo-diff-drive-system.so"
-        name="ignition::gazebo::systems::DiffDrive">
-        <left_joint>wheel_left_joint</left_joint>
-        <right_joint>wheel_right_joint</right_joint>
-		<!-- オドメトリが合うように車輪間隔を調整．0.230 → 0.2506 m -->
-		<!-- 車輪の中央ではなく外側のエッジで接していると解釈できる．0.230 + 0.0206 = 0.2506 -->
-        <wheel_separation>0.2506</wheel_separation>
-        <wheel_radius>0.0350</wheel_radius>
-        <odom_publish_frequency>30</odom_publish_frequency>
-        <topic>cmd_vel</topic>
-        <odom_topic>odom</odom_topic>
-        <tf_topic>tf</tf_topic>
-        <frame_id>odom</frame_id>
-        <child_frame_id>base_footprint</child_frame_id>
-	    </plugin>
-	  </gazebo>
+    <ros2_control name="IgnitionSystem" type="system">
+      <hardware>
+        <plugin>ign_ros2_control/IgnitionSystem</plugin>
+      </hardware>
+      <joint name="wheel_left_joint">
+        <command_interface name="velocity">
+          <param name="min">-1</param>
+          <param name="max">1</param>
+        </command_interface>
+        <state_interface name="position"/>
+        <state_interface name="velocity"/>
+      </joint>
+      <joint name="wheel_right_joint">
+        <command_interface name="velocity">
+          <param name="min">-1</param>
+          <param name="max">1</param>
+        </command_interface>
+        <state_interface name="position"/>
+        <state_interface name="velocity"/>
+      </joint>
+    </ros2_control>
+    <gazebo>
+      <!-- Joint state publisher -->
+      <plugin filename="ign_ros2_control-system" name="ign_ros2_control::IgnitionROS2ControlPlugin">
+        <parameters>$(find kobuki_description)/config/diff_drive_controller_velocity.yaml</parameters>
+        <ros>
+          <remapping>/diff_drive_base_controller/cmd_vel_unstamped:=/cmd_vel</remapping>
+        </ros>
+      </plugin>
+    </gazebo>
   </xacro:macro>
 </robot>

Commit message: ign_ros2_controlからlibignition-gazebo-diff-driveに戻す

File: kobuki_description/urdf/kobuki_gazebo.urdf.xacro (robot description, xacro)
@@ -144,34 +144,22 @@
       </sensor>
 	  </gazebo>
-    <ros2_control name="IgnitionSystem" type="system">
-      <hardware>
-        <plugin>ign_ros2_control/IgnitionSystem</plugin>
-      </hardware>
-      <joint name="wheel_left_joint">
-        <command_interface name="velocity">
-          <param name="min">-1</param>
-          <param name="max">1</param>
-        </command_interface>
-        <state_interface name="position"/>
-        <state_interface name="velocity"/>
-      </joint>
-      <joint name="wheel_right_joint">
-        <command_interface name="velocity">
-          <param name="min">-1</param>
-          <param name="max">1</param>
-        </command_interface>
-        <state_interface name="position"/>
-        <state_interface name="velocity"/>
-      </joint>
-    </ros2_control>
-    <gazebo>
-      <!-- Joint state publisher -->
-      <plugin filename="ign_ros2_control-system" name="ign_ros2_control::IgnitionROS2ControlPlugin">
-        <parameters>$(find kobuki_description)/config/diff_drive_controller_velocity.yaml</parameters>
-        <ros>
-          <remapping>/diff_drive_base_controller/cmd_vel_unstamped:=/cmd_vel</remapping>
-        </ros>
-      </plugin>
-    </gazebo>
+	  <gazebo>
+      <plugin
+        filename="libignition-gazebo-diff-drive-system.so"
+        name="ignition::gazebo::systems::DiffDrive">
+        <left_joint>wheel_left_joint</left_joint>
+        <right_joint>wheel_right_joint</right_joint>
+		<!-- オドメトリが合うように車輪間隔を調整．0.230 → 0.2506 m -->
+		<!-- 車輪の中央ではなく外側のエッジで接していると解釈できる．0.230 + 0.0206 = 0.2506 -->
+        <wheel_separation>0.2506</wheel_separation>
+        <wheel_radius>0.0350</wheel_radius>
+        <odom_publish_frequency>30</odom_publish_frequency>
+        <topic>cmd_vel</topic>
+        <odom_topic>odom</odom_topic>
+        <tf_topic>tf</tf_topic>
+        <frame_id>odom</frame_id>
+        <child_frame_id>base_footprint</child_frame_id>
+	    </plugin>
+	  </gazebo>
   </xacro:macro>
 </robot>
