Commit message: オドメトリがうまく行くように調整

File: kobuki_description/urdf/kobuki.urdf.xacro (robot description, xacro)
@@ -76,4 +76,55 @@
       </collision>
       <inertial>
+        <!-- 慣性を1kg（元の100倍）にしないとオドメトリが実際よりも大きくなる（車輪が空転している？） -->
+        <!-- 現実的な値ではないので，要改善 -->
+        <mass value="1.00" />
+        <origin xyz="0 0 0" />
+        <inertia ixx="3.42e-4" ixy="0.0" ixz="0.0"
+                 iyy="3.42e-4" iyz="0.0"
+                 izz="6.13e-4" />
+      </inertial>
+    </link>
+    <joint name="wheel_right_joint" type="continuous">
+      <parent link="base_link"/>
+      <child link="wheel_right_link"/>
+      <origin xyz="0.00 -${0.23/2} 0.0250" rpy="${-M_PI/2} 0 0"/>
+      <axis xyz="0 0 1"/>
+    </joint>
+    <link name="wheel_right_link">
+      <visual>
+        <geometry>
+          <mesh filename="file://$(find kobuki_description)/meshes/wheel.dae"/>
+        </geometry>
+        <origin xyz="0 0 0" rpy="0 0 0"/>
+      </visual>
+      <collision>
+        <geometry>
+          <cylinder length="0.0206" radius="0.035"/>
+        </geometry>
+        <origin rpy="0 0 0" xyz="0 0 0"/>
+      </collision>
+      <inertial>
+        <!-- 慣性を1kg（元の100倍）にしないとオドメトリが実際よりも大きくなる（車輪が空転している？） -->
+        <!-- 現実的な値ではないので，要改善 -->
+        <mass value="1.00" />
+        <origin xyz="0 0 0" />
+        <inertia ixx="3.42e-4" ixy="0.0" ixz="0.0"
+                 iyy="3.42e-4" iyz="0.0"
+                 izz="6.13e-4" />
+      </inertial>
+    </link>
+    <joint name="caster_front_joint" type="fixed">
+      <parent link="base_link"/>
+      <child link="caster_front_link"/>
+      <origin xyz="0.115 0.0 0.007" rpy="${-M_PI/2} 0 0"/>
+    </joint>
+    <link name="caster_front_link">
+      <collision>
+        <geometry>
+          <cylinder length="0.0176" radius="0.017"/>
+        </geometry>
+        <origin rpy="0 0 0" xyz="0 0 0"/>
+      </collision>
+      <inertial>
         <mass value="0.01" />
         <origin xyz="0 0 0" />
@@ -83,55 +134,8 @@
       </inertial>
     </link>
-    <joint name="wheel_right_joint" type="continuous">
-      <parent link="base_link"/>
-      <child link="wheel_right_link"/>
-      <origin xyz="0.00 -${0.23/2} 0.0250" rpy="${-M_PI/2} 0 0"/>
-      <axis xyz="0 0 1"/>
-    </joint>
-    <link name="wheel_right_link">
-      <visual>
-        <geometry>
-          <mesh filename="file://$(find kobuki_description)/meshes/wheel.dae"/>
-        </geometry>
-        <origin xyz="0 0 0" rpy="0 0 0"/>
-      </visual>
-      <collision>
-        <geometry>
-          <cylinder length="0.0206" radius="0.035"/>
-        </geometry>
-        <origin rpy="0 0 0" xyz="0 0 0"/>
-      </collision>
-      <inertial>
-        <mass value="0.01" />
-        <origin xyz="0 0 0" />
-        <inertia ixx="0.001" ixy="0.0" ixz="0.0"
-                 iyy="0.001" iyz="0.0"
-                 izz="0.001" />
-      </inertial>
-    </link>
-    <joint name="caster_front_joint" type="fixed">
-      <parent link="base_link"/>
-      <child link="caster_front_link"/>
-      <origin xyz="0.115 0.0 0.007" rpy="${-M_PI/2} 0 0"/>
-    </joint>
-    <link name="caster_front_link">
-      <collision>
-        <geometry>
-          <cylinder length="0.0176" radius="0.017"/>
-        </geometry>
-        <origin rpy="0 0 0" xyz="0 0 0"/>
-      </collision>
-      <inertial>
-        <mass value="0.01" />
-        <origin xyz="0 0 0" />
-        <inertia ixx="0.001" ixy="0.0" ixz="0.0"
-                 iyy="0.001" iyz="0.0"
-                 izz="0.001" />
-      </inertial>
-    </link>
     <joint name="caster_back_joint" type="fixed">
       <parent link="base_link"/>
       <child link="caster_back_link"/>
-      <origin xyz="-0.135 0.0 0.009" rpy="${-M_PI/2} 0 0"/>
+      <origin xyz="-0.135 0.0 0.0072" rpy="${-M_PI/2} 0 0"/>
     </joint>
     <link name="caster_back_link">

File: kobuki_description/urdf/kobuki_gazebo.urdf.xacro (robot description, xacro)
@@ -5,16 +5,16 @@
 	    <mu1>1.0</mu1>
 	    <mu2>1.0</mu2>
-	    <kp>1000000.0</kp>
-	    <kd>100.0</kd>
-	    <minDepth>0.001</minDepth>
-	    <maxVel>1.0</maxVel>
+	    <kp>1e+13</kp>
+	    <kd>1.0</kd>
+	    <minDepth>0.0001</minDepth>
+	    <maxVel>0.01</maxVel>
 	  </gazebo>
 	  <gazebo reference="wheel_right_link">
 	    <mu1>1.0</mu1>
 	    <mu2>1.0</mu2>
-	    <kp>1000000.0</kp>
-	    <kd>100.0</kd>
-	    <minDepth>0.001</minDepth>
-	    <maxVel>1.0</maxVel>
+	    <kp>1e+13</kp>
+	    <kd>1.0</kd>
+	    <minDepth>0.0001</minDepth>
+	    <maxVel>0.01</maxVel>
 	  </gazebo>
 	  <gazebo reference="caster_front_link">
@@ -150,6 +150,8 @@
         <left_joint>wheel_left_joint</left_joint>
         <right_joint>wheel_right_joint</right_joint>
-        <wheel_separation>0.230</wheel_separation>
-        <wheel_radius>0.035</wheel_radius>
+		<!-- オドメトリが合うように車輪間隔を調整．0.230 → 0.2506 m -->
+		<!-- 車輪の中央ではなく外側のエッジで接していると解釈できる．0.230 + 0.0206 = 0.2506 -->
+        <wheel_separation>0.2506</wheel_separation>
+        <wheel_radius>0.0350</wheel_radius>
         <odom_publish_frequency>30</odom_publish_frequency>
         <topic>cmd_vel</topic>

Commit message: OMXを搭載してもガタつかないようにオドメトリが正確になるように車輪を10kgに変更．

File: kobuki_description/urdf/kobuki.urdf.xacro (robot description, xacro)
@@ -76,11 +76,12 @@
       </collision>
       <inertial>
-        <!-- 慣性を1kg（元の100倍）にしないとオドメトリが実際よりも大きくなる（車輪が空転している？） -->
+        <!-- 慣性を10kg（元の1000倍）にしないとオドメトリが実際よりも大きくなる（車輪が空転している？） -->
+        <!-- OMXを搭載した場合は，1kgからさらに10kgにしないと安定に走行しない． -->
         <!-- 現実的な値ではないので，要改善 -->
-        <mass value="1.00" />
-        <origin xyz="0 0 0" />
-        <inertia ixx="3.42e-4" ixy="0.0" ixz="0.0"
-                 iyy="3.42e-4" iyz="0.0"
-                 izz="6.13e-4" />
+        <mass value="10.0" />
+        <origin xyz="0 0 0" />
+        <inertia ixx="3.42e-3" ixy="0.0" ixz="0.0"
+                 iyy="3.42e-3" iyz="0.0"
+                 izz="6.13e-3" />
       </inertial>
     </link>
@@ -105,11 +106,12 @@
       </collision>
       <inertial>
-        <!-- 慣性を1kg（元の100倍）にしないとオドメトリが実際よりも大きくなる（車輪が空転している？） -->
+        <!-- 慣性を10kg（元の1000倍）にしないとオドメトリが実際よりも大きくなる（車輪が空転している？） -->
+        <!-- OMXを搭載した場合は，1kgからさらに10kgにしないと安定に走行しない． -->
         <!-- 現実的な値ではないので，要改善 -->
-        <mass value="1.00" />
-        <origin xyz="0 0 0" />
-        <inertia ixx="3.42e-4" ixy="0.0" ixz="0.0"
-                 iyy="3.42e-4" iyz="0.0"
-                 izz="6.13e-4" />
+        <mass value="10.0" />
+        <origin xyz="0 0 0" />
+        <inertia ixx="3.42e-3" ixy="0.0" ixz="0.0"
+                 iyy="3.42e-3" iyz="0.0"
+                 izz="6.13e-3" />
       </inertial>
     </link>

Commit message: 車輪の慣性を1000倍にしていたのを戻した

File: kobuki_description/urdf/kobuki.urdf.xacro (robot description, xacro)
@@ -76,12 +76,9 @@
       </collision>
       <inertial>
-        <!-- 慣性を10kg（元の1000倍）にしないとオドメトリが実際よりも大きくなる（車輪が空転している？） -->
-        <!-- OMXを搭載した場合は，1kgからさらに10kgにしないと安定に走行しない． -->
-        <!-- 現実的な値ではないので，要改善 -->
-        <mass value="10.0" />
-        <origin xyz="0 0 0" />
-        <inertia ixx="3.42e-3" ixy="0.0" ixz="0.0"
-                 iyy="3.42e-3" iyz="0.0"
-                 izz="6.13e-3" />
+        <mass value="0.01" />
+        <origin xyz="0 0 0" />
+        <inertia ixx="3.42e-6" ixy="0.0" ixz="0.0"
+                 iyy="3.42e-6" iyz="0.0"
+                 izz="6.13e-6" />
       </inertial>
     </link>
@@ -106,12 +103,9 @@
       </collision>
       <inertial>
-        <!-- 慣性を10kg（元の1000倍）にしないとオドメトリが実際よりも大きくなる（車輪が空転している？） -->
-        <!-- OMXを搭載した場合は，1kgからさらに10kgにしないと安定に走行しない． -->
-        <!-- 現実的な値ではないので，要改善 -->
-        <mass value="10.0" />
-        <origin xyz="0 0 0" />
-        <inertia ixx="3.42e-3" ixy="0.0" ixz="0.0"
-                 iyy="3.42e-3" iyz="0.0"
-                 izz="6.13e-3" />
+        <mass value="0.01" />
+        <origin xyz="0 0 0" />
+        <inertia ixx="3.42e-6" ixy="0.0" ixz="0.0"
+                 iyy="3.42e-6" iyz="0.0"
+                 izz="6.13e-6" />
       </inertial>
     </link>
